File: Book Images/_autosave-_autosave-Book Images.sch (KiCad schematic (older format))
At the start: 27 parts, among them J1 7V to 20V, Q1 2N3904, Q2 TIP41, T1 4:1, U1 L7805, U1 NE555DR

Commit message: may 16
Parts:
- removed F1: 100mA, digikey-footprints:1206, symbol dk_Fuses:3413_0332_22
- added D5: GRN, symbol Device:LED_Small_ALT
- added R1: 560, symbol Device:R_Small_US
- added SW1: SW_SPST, symbol Switch:SW_SPST
- C1: value 10uF -> 470uF
- C2: value 10uF -> 47uF
- J1: value 7V to 20V -> 6V to 35V
- renumbered Vout to 5V_out
Connections:
- wire segments 59 -> 58
Other:
- moved on the sheet: BT1, C1, C2, D1, D2, D3, D4, J1, U1
